File: hardware/board/harp.device.valve-controller/isolated_usb_rp2040.kicad_sch (KiCad schematic)
At the start: 50 parts, among them J2 Conn_01x03_Male, J21 Conn_01x03_Male, J4 AudioJack3, J5 USB_C_Receptacle_USB2.0, U2 TPD2EUSB30, U3 ADUM4160, U4 RP2040, U5 W25Q16JVUXIQ, X1 ECS-TXO-2016

Commit message: add soft start ic; add status LEDs per output
Parts:
- FID1, FID2, FID3: now not fitted
Connections:
- net AUX_LED_ENABLE: now reaches U4.6 (GPIO4)
- no-connect marks 7 -> 6
Changed lines of the file:
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@@
 	)
 	(no_connect
-		(at 224.79 85.09)
-	)
-	(no_connect
 		(at 41.275 52.705)
 	)
@@
 	(wire
 		(pts
+			(xy 224.79 85.09) (xy 227.33 85.09)
+		)
+		(stroke
+			(width 0)
+			(type default)
+		)
+	)
+	(wire
+		(pts
 			(xy 24.13 86.995) (xy 25.4 86.995)
 		)
@@
 	(label "HARP_CLK_SYNC"
 		(at 40.64 123.825 0)
-		(fields_autoplaced yes)
 		(effects
 			(font
@@
 	(label "QSPI_CS"
 		(at 53.34 103.505 0)
-		(fields_autoplaced yes)
 		(effects
 			(font
@@
 	(label "UART0_TXD"
 		(at 227.33 74.93 0)
-		(fields_autoplaced yes)
 		(effects
 			(font
@@
 	(label "QSPI_D3"
 		(at 160.02 87.63 180)
-		(fields_autoplaced yes)
 		(effects
 			(font
@@
 	(label "QSPI_D2"
 		(at 160.02 85.09 180)
-		(fields_autoplaced yes)
 		(effects
 			(font
@@
 	(label "D-"
 		(at 95.25 41.91 180)
-		(fields_autoplaced yes)
 		(effects
 			(font
@@
 	(label "UART0_RXD"
 		(at 25.4 89.535 0)
-		(fields_autoplaced yes)
 		(effects
 			(font
@@
 	(label "QSPI_D1"
 		(at 160.02 82.55 180)
-		(fields_autoplaced yes)
 		(effects
 			(font
@@
 	(label "QSPI_D0"
 		(at 273.05 31.75 0)
-		(fields_autoplaced yes)
 		(effects
 			(font
@@
 	(label "DD-"
 		(at 146.05 41.91 0)
-		(fields_autoplaced yes)
 		(effects
 			(font
@@
 	(label "QSPI_D3"
 		(at 273.05 41.91 0)
-		(fields_autoplaced yes)
 		(effects
 			(font
@@
 	(label "DD+"
 		(at 146.05 39.37 0)
-		(fields_autoplaced yes)
 		(effects
 			(font
@@
 	(label "HARP_CLK_SYNC"
 		(at 227.33 87.63 0)
-		(fields_autoplaced yes)
 		(effects
 			(font
@@
 	(label "QSPI_CS"
 		(at 241.3 34.29 180)
-		(fields_autoplaced yes)
 		(effects
 			(font
@@
 	(label "USB_Boot"
 		(at 31.75 103.505 0)
-		(fields_autoplaced yes)
 		(effects
 			(font
@@
 	(label "UART0_TXD"
 		(at 25.4 86.995 0)
-		(fields_autoplaced yes)
 		(effects
 			(font
@@
 	(label "QSPI_CLK"
 		(at 241.3 39.37 180)
-		(fields_autoplaced yes)
 		(effects
 			(font
@@
 	(label "DD-"
 		(at 234.95 67.31 0)
-		(fields_autoplaced yes)
 		(effects
 			(font
@@
 	(label "UART0_RXD"
 		(at 227.33 77.47 0)
-		(fields_autoplaced yes)
 		(effects
 			(font
@@
 	(label "D-"
 		(at 68.58 38.735 0)
-		(fields_autoplaced yes)
 		(effects
 			(font
@@
 	(label "QSPI_D2"
 		(at 273.05 39.37 0)
-		(fields_autoplaced yes)
 		(effects
 			(font
@@
 	(label "VDD1"
 		(at 106.68 30.48 180)
-		(fields_autoplaced yes)
 		(effects
 			(font
@@
 	(label "VDD1"
 		(at 39.37 140.335 180)
-		(fields_autoplaced yes)
 		(effects
 			(font
@@
 	(label "D+"
 		(at 68.58 43.815 0)
-		(fields_autoplaced yes)
 		(effects
 			(font
@@
 	(label "D+"
 		(at 95.25 39.37 180)
-		(fields_autoplaced yes)
 		(effects
 			(font
@@
 	(label "QSPI_D1"
 		(at 273.05 34.29 0)
-		(fields_autoplaced yes)
 		(effects
 			(font
@@
 	(label "QSPI_D0"
 		(at 160.02 80.01 180)
-		(fields_autoplaced yes)
 		(effects
 			(font
@@
 	(label "QSPI_CLK"
 		(at 160.02 91.44 180)
-		(fields_autoplaced yes)
 		(effects
 			(font
@@
 	(label "QSPI_CS"
 		(at 160.02 76.2 180)
-		(fields_autoplaced yes)
 		(effects
 			(font
@@
 	(label "DD+"
 		(at 234.95 64.77 0)
-		(fields_autoplaced yes)
 		(effects
 			(font
@@
 		(shape input)
 		(at 227.33 92.71 0)
-		(fields_autoplaced yes)
 		(effects
 			(font
@@
 		(shape input)
 		(at 227.33 102.87 0)
-		(fields_autoplaced yes)
 		(effects
 			(font
@@
 		(shape input)
 		(at 227.33 118.11 0)
-		(fields_autoplaced yes)
 		(effects
 			(font
@@
 		(shape input)
 		(at 227.33 120.65 0)
-		(fields_autoplaced yes)
 		(effects
 			(font
@@
 		(shape input)
 		(at 227.33 123.19 0)
-		(fields_autoplaced yes)
 		(effects
 			(font
@@
 		(shape input)
 		(at 227.33 125.73 0)
-		(fields_autoplaced yes)
 		(effects
 			(font
@@
 		(shape input)
 		(at 227.33 128.27 0)
-		(fields_autoplaced yes)
 		(effects
 			(font
@@
 		(shape input)
 		(at 227.33 107.95 0)
-		(fields_autoplaced yes)
+		(effects
+			(font
+				(size 1.27 1.27)
+			)
+			(justify left)
+		)
+	)
+	(hierarchical_label "AUX_LED_ENABLE"
+		(shape input)
+		(at 227.33 85.09 0)
 		(effects
 			(font
@@
 		(shape input)
 		(at 227.33 95.25 0)
-		(fields_autoplaced yes)
 		(effects
 			(font
@@
 		(shape input)
 		(at 227.33 133.35 0)
-		(fields_autoplaced yes)
 		(effects
 			(font
@@
 		(shape input)
 		(at 227.33 143.51 0)
-		(fields_autoplaced yes)
 		(effects
 			(font
@@
 		(shape input)
 		(at 227.33 135.89 0)
-		(fields_autoplaced yes)
 		(effects
 			(font
@@
 		(shape input)
 		(at 227.33 146.05 0)
-		(fields_autoplaced yes)
 		(effects
 			(font
@@
 		(shape input)
 		(at 227.33 110.49 0)
-		(fields_autoplaced yes)
 		(effects
 			(font
@@
 		(shape input)
 		(at 227.33 138.43 0)
-		(fields_autoplaced yes)
 		(effects
 			(font
@@
 		(shape input)
 		(at 227.33 148.59 0)
-		(fields_autoplaced yes)
 		(effects
 			(font
@@
 		(shape input)
 		(at 227.33 90.17 0)
-		(fields_autoplaced yes)
 		(effects
 			(font
@@
 		(shape input)
 		(at 227.33 130.81 0)
-		(fields_autoplaced yes)
 		(effects
 			(font
@@
 		(shape input)
 		(at 227.33 105.41 0)
-		(fields_autoplaced yes)
 		(effects
 			(font
@@
 		(shape input)
 		(at 227.33 100.33 0)
-		(fields_autoplaced yes)
 		(effects
 			(font
@@
 		(shape input)
 		(at 227.33 113.03 0)
-		(fields_autoplaced yes)
 		(effects
 			(font
@@
 		(shape input)
 		(at 227.33 97.79 0)
-		(fields_autoplaced yes)
 		(effects
 			(font
@@
 		(shape input)
 		(at 227.33 151.13 0)
-		(fields_autoplaced yes)
 		(effects
 			(font
@@
 		(shape input)
 		(at 227.33 115.57 0)
-		(fields_autoplaced yes)
 		(effects
 			(font
@@
 		(in_bom yes)
 		(on_board yes)
-		(dnp no)
+		(dnp yes)
 		(property "Reference" "FID1"
 			(at 266.7 160.655 0)
@@
 		(in_bom yes)
 		(on_board yes)
-		(dnp no)
+		(dnp yes)
 		(property "Reference" "FID2"
 			(at 272.415 160.655 0)
@@
 		(in_bom yes)
 		(on_board yes)
-		(dnp no)
+		(dnp yes)
 		(property "Reference" "FID3"
 			(at 278.13 160.655 0)
