File: hardware/board/harp.device.valve-controller/valve-controller.kicad_pcb (KiCad board)
At the start: 4 copper layers, 70 x 168 mm, 185 parts, among them J1 Screw_Terminal_01x02, J10 Screw_Terminal_01x02, J11 Screw_Terminal_01x02, J12 Screw_Terminal_01x02, J13 Screw_Terminal_01x02, J14 Screw_Terminal_01x02, J15 Screw_Terminal_01x02, J16 Screw_Terminal_01x02, J17 Screw_Terminal_01x02, J18 Screw_Terminal_01x02, J19 Screw_Terminal_01x02, J2 Conn_01x03_Male, J20 Screw_Terminal_01x02, J21 Conn_01x03_Male, J26 Conn_02x10_Odd_Even, J3 Screw_Terminal_01x02, J4 AudioJack3, J5 USB_C_Receptacle_USB2.0, J6 Screw_Terminal_01x02, J7 Screw_Terminal_01x02, J8 Screw_Terminal_01x02, J9 Screw_Terminal_01x02, Q1 CSD17570Q5B, Q10 CSD17570Q5B, Q11 CSD17570Q5B, Q12 CSD17570Q5B, Q13 CSD17570Q5B, Q14 CSD17570Q5B, Q15 CSD17570Q5B, Q16 CSD17570Q5B, Q17 CSD17570Q5B, Q2 GSFD4005, Q3 CSD17570Q5B, Q4 CSD17570Q5B, Q5 CSD17570Q5B, Q6 CSD17570Q5B, Q7 CSD17570Q5B, Q8 CSD17570Q5B, Q9 CSD17570Q5B, U1 MIC4127, U10 MIC4127, U11 MIC4127, U12 MIC4127, U13 MIC4127, U14 MIC4127, U15 LMR51430, U2 TPD2EUSB30, U3 ADUM4160, U4 RP2040, U5 W25Q16JVUXIQ, U6 MIC4127, U7 rt6150b-33gqw, U8 MIC4127, X1 ECS-TXO-2016

Commit message: add soft start ic; add status LEDs per output
Parts:
- added D22: LED, LED_SMD:LED_0603_1608Metric_Pad1.05x0.95mm_HandSolder, F.Cu at (83.5, 23.8)
- added D23: LED, LED_SMD:LED_0603_1608Metric_Pad1.05x0.95mm_HandSolder, F.Cu at (83.5, 33.5)
- added D24: LED, LED_SMD:LED_0603_1608Metric_Pad1.05x0.95mm_HandSolder, F.Cu at (83.5, 43.3)
- added D25: LED, LED_SMD:LED_0603_1608Metric_Pad1.05x0.95mm_HandSolder, F.Cu at (83.5, 53.0)
- added D26: LED, LED_SMD:LED_0603_1608Metric_Pad1.05x0.95mm_HandSolder, F.Cu at (83.5, 62.7)
- added D27: LED, LED_SMD:LED_0603_1608Metric_Pad1.05x0.95mm_HandSolder, F.Cu at (83.5, 72.5)
- added D28: LED, LED_SMD:LED_0603_1608Metric_Pad1.05x0.95mm_HandSolder, F.Cu at (83.5, 82.2)
- added D29: LED, LED_SMD:LED_0603_1608Metric_Pad1.05x0.95mm_HandSolder, F.Cu at (83.5, 91.9)
- added D30: LED, LED_SMD:LED_0603_1608Metric_Pad1.05x0.95mm_HandSolder, F.Cu at (83.5, 101.7)
- added D31: LED, LED_SMD:LED_0603_1608Metric_Pad1.05x0.95mm_HandSolder, F.Cu at (83.5, 111.4)
- added D32: LED, LED_SMD:LED_0603_1608Metric_Pad1.05x0.95mm_HandSolder, F.Cu at (83.5, 121.1)
- added D33: LED, LED_SMD:LED_0603_1608Metric_Pad1.05x0.95mm_HandSolder, F.Cu at (83.5, 130.9)
- added D34: LED, LED_SMD:LED_0603_1608Metric_Pad1.05x0.95mm_HandSolder, F.Cu at (83.5, 140.6)
- added D35: LED, LED_SMD:LED_0603_1608Metric_Pad1.05x0.95mm_HandSolder, F.Cu at (83.5, 150.3)
- added D36: LED, LED_SMD:LED_0603_1608Metric_Pad1.05x0.95mm_HandSolder, F.Cu at (83.5, 160.1)
- added D37: LED, LED_SMD:LED_0603_1608Metric_Pad1.05x0.95mm_HandSolder, F.Cu at (83.5, 169.8)
- added Q18: SUD19P06-60L-E3, Package_TO_SOT_SMD:TO-252-2, F.Cu at (117.0, 30.1)
- added Q20: 2N7002, Package_TO_SOT_SMD:SOT-23, F.Cu at (98.5, 81.2)
- added R19: 100K, Resistor_SMD:R_0402_1005Metric, F.Cu at (116.8, 47.0)
- added R20: 39K2, Resistor_SMD:R_0402_1005Metric, F.Cu at (116.8, 48.0)
- added R52: 100K, Resistor_SMD:R_0402_1005Metric, F.Cu at (119.2, 38.7)
- added R53: 1K6, Resistor_SMD:R_0402_1005Metric, F.Cu at (98.3, 28.6)
- added R54: 1K6, Resistor_SMD:R_0402_1005Metric, F.Cu at (98.3, 35.2)
- added R55: 1K6, Resistor_SMD:R_0402_1005Metric, F.Cu at (98.3, 48.0)
- added R56: 1K6, Resistor_SMD:R_0402_1005Metric, F.Cu at (98.3, 54.6)
- added R57: 1K6, Resistor_SMD:R_0402_1005Metric, F.Cu at (98.3, 67.5)
- added R58: 1K6, Resistor_SMD:R_0402_1005Metric, F.Cu at (98.3, 74.1)
- added R59: 1K6, Resistor_SMD:R_0402_1005Metric, F.Cu at (98.3, 86.9)
- added R60: 1K6, Resistor_SMD:R_0402_1005Metric, F.Cu at (98.3, 93.5)
- added R61: 1K6, Resistor_SMD:R_0402_1005Metric, F.Cu at (98.3, 106.4)
- added R62: 1K6, Resistor_SMD:R_0402_1005Metric, F.Cu at (98.3, 113.0)
- added R63: 1K6, Resistor_SMD:R_0402_1005Metric, F.Cu at (98.3, 125.9)
- added R64: 1K6, Resistor_SMD:R_0402_1005Metric, F.Cu at (98.3, 132.5)
- added R65: 1K6, Resistor_SMD:R_0402_1005Metric, F.Cu at (98.3, 145.4)
- added R66: 1K6, Resistor_SMD:R_0402_1005Metric, F.Cu at (98.3, 152.0)
- added R67: 1K6, Resistor_SMD:R_0402_1005Metric, F.Cu at (98.3, 164.8)
- added R68: 1K6, Resistor_SMD:R_0402_1005Metric, F.Cu at (98.3, 171.4)
- added R69: 10K, Resistor_SMD:R_0402_1005Metric, F.Cu at (100.8, 81.1)
- added U9: ~, Package_TO_SOT_SMD:SOT-23-6, F.Cu at (117.0, 38.7)
- moved C52 3.11 mm to (120.0, 44.8)
- moved U15 2.88 mm to (119.9, 47.0)
- moved C51 2.88 mm to (120.0, 49.4)
- moved L1 2.70 mm to (129.8, 47.0)
- moved C46 2.70 mm to (138.5, 45.0)
- moved C47 2.70 mm to (138.5, 47.0)
- moved C48 2.70 mm to (138.5, 49.0)
- moved R50 2.53 mm to (116.2, 45.5)
- moved R51 2.53 mm to (117.2, 45.5)
- moved C50 2.24 mm to (119.9, 42.1)
- moved C11 0.25 mm to (101.0, 104.0)
- moved D7 0.20 mm to (83.0, 46.4)
- moved C14 0.20 mm to (115.8, 98.9)
- moved C18 0.20 mm to (115.8, 97.9)
- moved C7 0.20 mm to (115.8, 96.9)
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Connections:
- net /Harp Core RP2040 + Isolated USB/OUT0 renamed /OUT0
- net /Harp Core RP2040 + Isolated USB/OUT1 renamed /OUT1
- net /Harp Core RP2040 + Isolated USB/OUT10 renamed /OUT10
- net /Harp Core RP2040 + Isolated USB/OUT11 renamed /OUT11
- net /Harp Core RP2040 + Isolated USB/OUT12 renamed /OUT12
- net /Harp Core RP2040 + Isolated USB/OUT13 renamed /OUT13
- net /Harp Core RP2040 + Isolated USB/OUT14 renamed /OUT14
- net /Harp Core RP2040 + Isolated USB/OUT15 renamed /OUT15
- net /Harp Core RP2040 + Isolated USB/OUT2 renamed /OUT2
- net /Harp Core RP2040 + Isolated USB/OUT3 renamed /OUT3
- net /Harp Core RP2040 + Isolated USB/OUT4 renamed /OUT4
- net /Harp Core RP2040 + Isolated USB/OUT5 renamed /OUT5
- net /Harp Core RP2040 + Isolated USB/OUT6 renamed /OUT6
- net /Harp Core RP2040 + Isolated USB/OUT7 renamed /OUT7
- net /Harp Core RP2040 + Isolated USB/OUT8 renamed /OUT8
- net /Harp Core RP2040 + Isolated USB/OUT9 renamed /OUT9
- U15 pad 5: VPP -> Net-(U15-EN)
- U4 pad 6: unconnected-(U4-GPIO4-Pad6) -> /AUX_LED_ENABLE
Routing:
- net /LED_ENABLE_MOSFET_D: track 0.00 -> 67.9 mm, vias 0 -> 17
- net VPP: track 79.5 -> 108.6 mm, vias 9 -> 16
- net /AUX_LED_ENABLE: track 0.00 -> 22.0 mm, vias 0 -> 2
- net Net-(D9-K): track 0.00 -> 18.7 mm
- net Net-(D34-A): track 0.00 -> 15.4 mm
- net Net-(D32-A): track 0.00 -> 15.4 mm
- net Net-(D26-A): track 0.00 -> 15.4 mm
- net Net-(D22-A): track 0.00 -> 15.4 mm
- net Net-(D36-A): track 0.00 -> 15.4 mm
- net Net-(D30-A): track 0.00 -> 15.4 mm
- net Net-(D28-A): track 0.00 -> 15.4 mm
- net Net-(D24-A): track 0.00 -> 15.4 mm
- net Net-(D35-A): track 0.00 -> 14.1 mm, vias 0 -> 2
- net Net-(D23-A): track 0.00 -> 14.1 mm, vias 0 -> 2
- net Net-(D25-A): track 0.00 -> 14.1 mm, vias 0 -> 2
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- added copper zone on In2.Cu, net /LED_ENABLE_MOSFET_D
Other:
- board text added: "0368-E-001-001.001.000"
- board text added: "9-24VDC 5A"
- board text added: "Sonya Vasquez Sept 9, 2025"
- board text removed: "0368-E-001-001.000.000"
- board text removed: "5-24VDC 5A"
- board text removed: "Sonya Vasquez Feb 11, 2025"
